Commit message: Adjusted ARMAR 4 model to support a floating base

File: armar/description/urdf/armar4_fixed_hands_and_legs.urdf (robot description, URDF)
Before this commit: robot main, 47 links, 46 joints
Links:
- removed link world
- added link base, mass 0.00001
Joints:
- joint root_joint: parent world -> base
